Commit message: Feat: Working AMCL

File: my_robot/urdf/my_robot.xacro (robot description, xacro)
@@ -2,8 +2,8 @@
 <robot name="my_robot" xmlns:xacro="http://www.ros.org/wiki/xacro">
   <xacro:include filename="$(find my_robot)/urdf/my_robot.gazebo" />
-  <link name="robot_footprint"></link>
+  <link name="base_link"></link>
   <joint name="robot_footprint_joint" type="fixed">
     <origin xyz="0 0 0" rpy="0 0 0" />
-    <parent link="robot_footprint"/>
+    <parent link="base_link"/>
     <child link="chassis" />
   </joint>

Commit message: fix: let hokuyo see over wheels and make robot turn more easily

File: my_robot/urdf/my_robot.xacro (robot description, xacro)
@@ -45,5 +45,5 @@
       <origin xyz="0 0 0" rpy="0 1.5707 1.5707"/>
       <geometry>
-        <cylinder radius="0.1" length="0.05"/>
+        <cylinder radius="0.06" length="0.05"/>
       </geometry>
     </collision>
@@ -51,5 +51,5 @@
       <origin xyz="0 0 0" rpy="0 1.5707 1.5707"/>
       <geometry>
-        <cylinder radius="0.1" length="0.05"/>
+        <cylinder radius="0.06" length="0.05"/>
       </geometry>
     </visual>
@@ -68,5 +68,5 @@
       <origin xyz="0 0 0" rpy="0 1.5707 1.5707"/>
       <geometry>
-        <cylinder radius="0.1" length="0.05"/>
+        <cylinder radius="0.06" length="0.05"/>
       </geometry>
     </collision>
@@ -74,5 +74,5 @@
       <origin xyz="0 0 0" rpy="0 1.5707 1.5707"/>
       <geometry>
-        <cylinder radius="0.1" length="0.05"/>
+        <cylinder radius="0.06" length="0.05"/>
       </geometry>
     </visual>
@@ -91,5 +91,5 @@
       <origin xyz="0 0 0" rpy="0 1.5707 1.5707"/>
       <geometry>
-        <cylinder radius="0.1" length="0.05"/>
+        <cylinder radius="0.06" length="0.05"/>
       </geometry>
     </collision>
@@ -97,5 +97,5 @@
       <origin xyz="0 0 0" rpy="0 1.5707 1.5707"/>
       <geometry>
-        <cylinder radius="0.1" length="0.05"/>
+        <cylinder radius="0.06" length="0.05"/>
       </geometry>
     </visual>
@@ -114,5 +114,5 @@
       <origin xyz="0 0 0" rpy="0 1.5707 1.5707"/>
       <geometry>
-        <cylinder radius="0.1" length="0.05"/>
+        <cylinder radius="0.06" length="0.05"/>
       </geometry>
     </collision>
@@ -120,10 +120,10 @@
       <origin xyz="0 0 0" rpy="0 1.5707 1.5707"/>
       <geometry>
-        <cylinder radius="0.1" length="0.05"/>
+        <cylinder radius="0.06" length="0.05"/>
       </geometry>
     </visual>
   </link>
   <joint type="continuous" name="front_left_wheel_hinge">
-    <origin xyz="0.15 0.15 0" rpy="0 0 0"/>
+    <origin xyz="0.08 0.13 0" rpy="0 0 0"/>
     <child link="front_left_wheel"/>
     <parent link="chassis"/>
@@ -133,5 +133,5 @@
   </joint>
   <joint type="continuous" name="front_right_wheel_hinge">
-    <origin xyz="0.15 -0.15 0" rpy="0 0 0"/>
+    <origin xyz="0.08 -0.13 0" rpy="0 0 0"/>
     <child link="front_right_wheel"/>
     <parent link="chassis"/>
@@ -141,5 +141,5 @@
   </joint>
   <joint type="continuous" name="rear_left_wheel_hinge">
-    <origin xyz="-0.15 0.15 0" rpy="0 0 0"/>
+    <origin xyz="-0.08 0.13 0" rpy="0 0 0"/>
     <child link="rear_left_wheel"/>
     <parent link="chassis"/>
@@ -149,5 +149,5 @@
   </joint>
   <joint type="continuous" name="rear_right_wheel_hinge">
-    <origin xyz="-0.15 -0.15 0" rpy="0 0 0"/>
+    <origin xyz="-0.08 -0.13 0" rpy="0 0 0"/>
     <child link="rear_right_wheel"/>
     <parent link="chassis"/>
@@ -215,5 +215,5 @@
   </link>
   <joint type="fixed" name="hokuyo_joint">
-    <origin xyz="0.15 0 0.1" rpy="0 0 0"/>
+    <origin xyz="0.0 0 0.08" rpy="0 0 0"/>
     <child link="hokuyo"/>
     <parent link="chassis"/>

Commit message: feature: map and localize with rtabmap

File: my_robot/urdf/my_robot.xacro (robot description, xacro)
@@ -156,5 +156,5 @@
     <dynamics damping="1.0" friction="1.0"/>
   </joint>
-  <link name='camera'>
+  <link name='camera_link'>
     <inertial>
       <mass value="0.1"/>
@@ -184,8 +184,15 @@
   <joint type="fixed" name="camera_joint">
     <origin xyz="0.2 0 0" rpy="0 0 0"/>
-    <child link="camera"/>
-    <parent link="chassis"/>
-    <axis xyz="0 1 0" rpy="0 0 0"/>
-  </joint>
+    <child link="camera_link"/>
+    <parent link="chassis"/>
+    <axis xyz="0 1 0" rpy="0 0 0"/>
+  </joint>
+  <joint name="camera_optical_joint" type="fixed">
+    <origin xyz="0 0 0" rpy="-1.5707 0 -1.5707"/>
+    <parent link="camera_link"/>
+    <child link="camera_link_optical"/>
+  </joint>
+  <link name="camera_link_optical">
+  </link>
   <link name='hokuyo'>
     <inertial>
